File: Eagle/Projet electronique - PIC-PIR - Groupe 5.sch (EAGLE design)
At the start: 13 parts, among them IC1 4511N, IC2 4511N

Commit message: update eagle file
Parts:
- added LED1, LED2: (no value), led:LED5MM
- added R3, R4: (no value), rcl:R-EU_0207/10
Connections:
- new net N$12: DIS1.A, IC1A.A
- new net N$13: DIS1.B, IC1A.B
- new net N$14: DIS1.C, IC1A.C
- new net N$15: DIS1.D, IC1A.D
- new net N$16: DIS1.E, IC1A.E
- new net N$17: DIS1.F, IC1A.F
- new net N$18: DIS1.G, IC1A.G
- new net N$19: DIS2.A, IC2A.A
- new net N$20: DIS2.B, IC2A.B
- new net N$21: DIS2.C, IC2A.C
- new net N$22: DIS2.D, IC2A.D
- new net N$23: DIS2.E, IC2A.E
- new net N$24: DIS2.F, IC2A.F
- new net N$25: DIS2.G, IC2A.G
- new net N$26: DIS1.CC, DIS1.CC@1, DIS2.CC, DIS2.CC@1, R3.1
- new net N$27: LED1.C, LED2.C, R4.2
- new net RE1: LED2.A, PIC.RE1/!WR/AN6
- new net RE2: LED1.A, PIC.RE2/!CS/AN7
- net GND: now also R3.2, R4.1
Other:
- moved on the sheet: DIS2
Changed lines of the file:
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@@
 <part name="DIS1" library="display-hp" library_urn="urn:adsk.eagle:library:212" deviceset="HD-H103" device="" package3d_urn="urn:adsk.eagle:package:13006/1"/>
 <part name="DIS2" library="display-hp" library_urn="urn:adsk.eagle:library:212" deviceset="HD-H103" device="" package3d_urn="urn:adsk.eagle:package:13006/1"/>
+<part name="R3" library="rcl" library_urn="urn:adsk.eagle:library:334" deviceset="R-EU_" device="0207/10" package3d_urn="urn:adsk.eagle:package:23491/2"/>
+<part name="LED1" library="led" library_urn="urn:adsk.eagle:library:259" deviceset="LED" device="5MM" package3d_urn="urn:adsk.eagle:package:15799/2"/>
+<part name="LED2" library="led" library_urn="urn:adsk.eagle:library:259" deviceset="LED" device="5MM" package3d_urn="urn:adsk.eagle:package:15799/2"/>
+<part name="R4" library="rcl" library_urn="urn:adsk.eagle:library:334" deviceset="R-EU_" device="0207/10" package3d_urn="urn:adsk.eagle:package:23491/2"/>
 </parts>
 <sheets>
@@
 <attribute name="VALUE" x="30.48" y="278.13" size="1.778" layer="96" rot="R180"/>
 </instance>
-<instance part="DIS2" gate="N" x="27.94" y="226.06" smashed="yes" rot="R90">
-<attribute name="NAME" x="33.02" y="216.535" size="1.778" layer="95" rot="R180"/>
-<attribute name="VALUE" x="33.02" y="237.49" size="1.778" layer="96" rot="R180"/>
+<instance part="DIS2" gate="N" x="27.94" y="228.6" smashed="yes" rot="R90">
+<attribute name="NAME" x="33.02" y="219.075" size="1.778" layer="95" rot="R180"/>
+<attribute name="VALUE" x="33.02" y="240.03" size="1.778" layer="96" rot="R180"/>
+</instance>
+<instance part="R3" gate="G$1" x="68.58" y="254" smashed="yes">
+<attribute name="NAME" x="64.77" y="255.4986" size="1.778" layer="95"/>
+<attribute name="VALUE" x="64.77" y="250.698" size="1.778" layer="96"/>
+</instance>
+<instance part="LED1" gate="G$1" x="-38.1" y="198.12" smashed="yes">
+<attribute name="NAME" x="-34.544" y="193.548" size="1.778" layer="95" rot="R90"/>
+<attribute name="VALUE" x="-32.385" y="193.548" size="1.778" layer="96" rot="R90"/>
+</instance>
+<instance part="LED2" gate="G$1" x="-25.4" y="198.12" smashed="yes">
+<attribute name="NAME" x="-21.844" y="193.548" size="1.778" layer="95" rot="R90"/>
+<attribute name="VALUE" x="-19.685" y="193.548" size="1.778" layer="96" rot="R90"/>
+</instance>
+<instance part="R4" gate="G$1" x="-30.48" y="175.26" smashed="yes" rot="R90">
+<attribute name="NAME" x="-31.9786" y="171.45" size="1.778" layer="95" rot="R90"/>
+<attribute name="VALUE" x="-27.178" y="171.45" size="1.778" layer="96" rot="R90"/>
 </instance>
 </instances>
@@
 <wire x1="-20.32" y1="243.84" x2="-17.78" y2="243.84" width="0.1524" layer="91"/>
 <label x="-17.78" y="243.84" size="1.778" layer="95"/>
+</segment>
+<segment>
+<pinref part="R3" gate="G$1" pin="2"/>
+<wire x1="73.66" y1="254" x2="78.74" y2="254" width="0.1524" layer="91"/>
+<label x="78.74" y="254" size="1.778" layer="95"/>
+</segment>
+<segment>
+<pinref part="R4" gate="G$1" pin="1"/>
+<wire x1="-30.48" y1="170.18" x2="-30.48" y2="167.64" width="0.1524" layer="91"/>
+<label x="-30.48" y="167.64" size="1.778" layer="95"/>
 </segment>
 </net>
@@
 </segment>
 </net>
+<net name="N$12" class="0">
+<segment>
+<pinref part="IC1" gate="A" pin="A"/>
+<pinref part="DIS1" gate="N" pin="A"/>
+<wire x1="-15.24" y1="274.32" x2="10.16" y2="274.32" width="0.1524" layer="91"/>
+</segment>
+</net>
+<net name="N$13" class="0">
+<segment>
+<pinref part="IC1" gate="A" pin="B"/>
+<pinref part="DIS1" gate="N" pin="B"/>
+<wire x1="-15.24" y1="271.78" x2="10.16" y2="271.78" width="0.1524" layer="91"/>
+</segment>
+</net>
+<net name="N$14" class="0">
+<segment>
+<pinref part="IC1" gate="A" pin="C"/>
+<pinref part="DIS1" gate="N" pin="C"/>
+<wire x1="-15.24" y1="269.24" x2="10.16" y2="269.24" width="0.1524" layer="91"/>
+</segment>
+</net>
+<net name="N$15" class="0">
+<segment>
+<pinref part="IC1" gate="A" pin="D"/>
+<pinref part="DIS1" gate="N" pin="D"/>
+<wire x1="-15.24" y1="266.7" x2="10.16" y2="266.7" width="0.1524" layer="91"/>
+</segment>
+</net>
+<net name="N$16" class="0">
+<segment>
+<pinref part="IC1" gate="A" pin="E"/>
+<pinref part="DIS1" gate="N" pin="E"/>
+<wire x1="-15.24" y1="264.16" x2="10.16" y2="264.16" width="0.1524" layer="91"/>
+</segment>
+</net>
+<net name="N$17" class="0">
+<segment>
+<pinref part="IC1" gate="A" pin="F"/>
+<pinref part="DIS1" gate="N" pin="F"/>
+<wire x1="-15.24" y1="261.62" x2="10.16" y2="261.62" width="0.1524" layer="91"/>
+</segment>
+</net>
+<net name="N$18" class="0">
+<segment>
+<pinref part="IC1" gate="A" pin="G"/>
+<pinref part="DIS1" gate="N" pin="G"/>
+<wire x1="-15.24" y1="259.08" x2="10.16" y2="259.08" width="0.1524" layer="91"/>
+</segment>
+</net>
+<net name="N$19" class="0">
+<segment>
+<pinref part="IC2" gate="A" pin="A"/>
+<pinref part="DIS2" gate="N" pin="A"/>
+<wire x1="-15.24" y1="236.22" x2="12.7" y2="236.22" width="0.1524" layer="91"/>
+</segment>
+</net>
+<net name="N$20" class="0">
+<segment>
+<pinref part="IC2" gate="A" pin="B"/>
+<pinref part="DIS2" gate="N" pin="B"/>
+<wire x1="-15.24" y1="233.68" x2="12.7" y2="233.68" width="0.1524" layer="91"/>
+</segment>
+</net>
+<net name="N$21" class="0">
+<segment>
+<pinref part="IC2" gate="A" pin="C"/>
+<pinref part="DIS2" gate="N" pin="C"/>
+<wire x1="-15.24" y1="231.14" x2="12.7" y2="231.14" width="0.1524" layer="91"/>
+</segment>
+</net>
+<net name="N$22" class="0">
+<segment>
+<pinref part="IC2" gate="A" pin="D"/>
+<pinref part="DIS2" gate="N" pin="D"/>
+<wire x1="-15.24" y1="228.6" x2="12.7" y2="228.6" width="0.1524" layer="91"/>
+</segment>
+</net>
+<net name="N$23" class="0">
+<segment>
+<pinref part="IC2" gate="A" pin="E"/>
+<pinref part="DIS2" gate="N" pin="E"/>
+<wire x1="-15.24" y1="226.06" x2="12.7" y2="226.06" width="0.1524" layer="91"/>
+</segment>
+</net>
+<net name="N$24" class="0">
+<segment>
+<pinref part="IC2" gate="A" pin="F"/>
+<pinref part="DIS2" gate="N" pin="F"/>
+<wire x1="-15.24" y1="223.52" x2="12.7" y2="223.52" width="0.1524" layer="91"/>
+</segment>
+</net>
+<net name="N$25" class="0">
+<segment>
+<pinref part="IC2" gate="A" pin="G"/>
+<pinref part="DIS2" gate="N" pin="G"/>
+<wire x1="-15.24" y1="220.98" x2="12.7" y2="220.98" width="0.1524" layer="91"/>
+</segment>
+</net>
+<net name="N$26" class="0">
+<segment>
+<pinref part="DIS1" gate="N" pin="CC@1"/>
+<wire x1="40.64" y1="274.32" x2="43.18" y2="274.32" width="0.1524" layer="91"/>
+<pinref part="DIS1" gate="N" pin="CC"/>
+<wire x1="43.18" y1="274.32" x2="43.18" y2="271.78" width="0.1524" layer="91"/>
+<wire x1="43.18" y1="271.78" x2="40.64" y2="271.78" width="0.1524" layer="91"/>
+<wire x1="43.18" y1="271.78" x2="55.88" y2="271.78" width="0.1524" layer="91"/>
+<junction x="43.18" y="271.78"/>
+<pinref part="DIS2" gate="N" pin="CC@1"/>
+<wire x1="43.18" y1="236.22" x2="45.72" y2="236.22" width="0.1524" layer="91"/>
+<pinref part="DIS2" gate="N" pin="CC"/>
+<wire x1="45.72" y1="236.22" x2="45.72" y2="233.68" width="0.1524" layer="91"/>
+<wire x1="45.72" y1="233.68" x2="43.18" y2="233.68" width="0.1524" layer="91"/>
+<wire x1="45.72" y1="236.22" x2="55.88" y2="236.22" width="0.1524" layer="91"/>
+<junction x="45.72" y="236.22"/>
+<wire x1="55.88" y1="271.78" x2="55.88" y2="254" width="0.1524" layer="91"/>
+<wire x1="55.88" y1="254" x2="55.88" y2="236.22" width="0.1524" layer="91"/>
+<wire x1="55.88" y1="254" x2="63.5" y2="254" width="0.1524" layer="91"/>
+<junction x="55.88" y="254"/>
+<pinref part="R3" gate="G$1" pin="1"/>
+</segment>
+</net>
+<net name="RE1" class="0">
+<segment>
+<pinref part="PIC" gate="G$1" pin="RE1/!WR/AN6"/>
+<wire x1="-119.38" y1="246.38" x2="-121.92" y2="246.38" width="0.1524" layer="91"/>
+<label x="-121.92" y="246.38" size="1.778" layer="95" rot="R180"/>
+</segment>
+<segment>
+<pinref part="LED2" gate="G$1" pin="A"/>
+<wire x1="-25.4" y1="200.66" x2="-25.4" y2="203.2" width="0.1524" layer="91"/>
+<label x="-25.4" y="203.2" size="1.778" layer="95" rot="R180"/>
+</segment>
+</net>
+<net name="RE2" class="0">
+<segment>
+<pinref part="PIC" gate="G$1" pin="RE2/!CS/AN7"/>
+<wire x1="-119.38" y1="243.84" x2="-121.92" y2="243.84" width="0.1524" layer="91"/>
+<label x="-121.92" y="243.84" size="1.778" layer="95" rot="R180"/>
+</segment>
+<segment>
+<pinref part="LED1" gate="G$1" pin="A"/>
+<wire x1="-38.1" y1="200.66" x2="-38.1" y2="203.2" width="0.1524" layer="91"/>
+<label x="-38.1" y="203.2" size="1.778" layer="95" rot="R180"/>
+</segment>
+</net>
+<net name="N$27" class="0">
+<segment>
+<pinref part="LED1" gate="G$1" pin="C"/>
+<wire x1="-38.1" y1="193.04" x2="-38.1" y2="187.96" width="0.1524" layer="91"/>
+<pinref part="LED2" gate="G$1" pin="C"/>
+<wire x1="-38.1" y1="187.96" x2="-33.02" y2="187.96" width="0.1524" layer="91"/>
+<wire x1="-30.48" y1="187.96" x2="-25.4" y2="187.96" width="0.1524" layer="91"/>
+<wire x1="-25.4" y1="187.96" x2="-25.4" y2="193.04" width="0.1524" layer="91"/>
+<wire x1="-33.02" y1="187.96" x2="-30.48" y2="187.96" width="0.1524" layer="91"/>
+<wire x1="-30.48" y1="187.96" x2="-30.48" y2="180.34" width="0.1524" layer="91"/>
+<pinref part="R4" gate="G$1" pin="2"/>
+</segment>
+</net>

Commit message: update file eagle
Parts:
- added X2: (no value), con-subd:F09H
Connections:
- new net RX: PIC.RX/RC7, X2.3
- new net TX: PIC.TX/RC6, X2.2
- net GND: now also X2.5
Changed lines of the file:
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@@
 <part name="LED2" library="led" library_urn="urn:adsk.eagle:library:259" deviceset="LED" device="5MM" package3d_urn="urn:adsk.eagle:package:15799/2"/>
 <part name="R4" library="rcl" library_urn="urn:adsk.eagle:library:334" deviceset="R-EU_" device="0207/10" package3d_urn="urn:adsk.eagle:package:23491/2"/>
+<part name="X2" library="con-subd" library_urn="urn:adsk.eagle:library:189" deviceset="F09" device="H" package3d_urn="urn:adsk.eagle:package:10276/1"/>
 </parts>
 <sheets>
@@
 <attribute name="NAME" x="-31.9786" y="171.45" size="1.778" layer="95" rot="R90"/>
 <attribute name="VALUE" x="-27.178" y="171.45" size="1.778" layer="96" rot="R90"/>
+</instance>
+<instance part="X2" gate="G$1" x="-76.2" y="193.04" smashed="yes">
+<attribute name="VALUE" x="-80.01" y="182.245" size="1.778" layer="96"/>
+<attribute name="NAME" x="-80.01" y="201.93" size="1.778" layer="95"/>
 </instance>
 </instances>
@@
 <wire x1="-30.48" y1="170.18" x2="-30.48" y2="167.64" width="0.1524" layer="91"/>
 <label x="-30.48" y="167.64" size="1.778" layer="95"/>
+</segment>
+<segment>
+<pinref part="X2" gate="G$1" pin="5"/>
+<wire x1="-83.82" y1="187.96" x2="-88.9" y2="187.96" width="0.1524" layer="91"/>
+<label x="-88.9" y="187.96" size="1.778" layer="95" rot="R180"/>
 </segment>
 </net>
@@
 <segment>
 <pinref part="IC1" gate="A" pin="IA"/>
-<wire x1="-40.64" y1="274.32" x2="-55.88" y2="274.32" width="0.1524" layer="91"/>
-<wire x1="-55.88" y1="274.32" x2="-55.88" y2="248.92" width="0.1524" layer="91"/>
+<wire x1="-40.64" y1="274.32" x2="-50.8" y2="274.32" width="0.1524" layer="91"/>
+<wire x1="-50.8" y1="274.32" x2="-50.8" y2="248.92" width="0.1524" layer="91"/>
 <pinref part="PIC" gate="G$1" pin="INT/RB0"/>
-<wire x1="-55.88" y1="248.92" x2="-76.2" y2="248.92" width="0.1524" layer="91"/>
+<wire x1="-50.8" y1="248.92" x2="-76.2" y2="248.92" width="0.1524" layer="91"/>
 </segment>
 </net>
@@
 <segment>
 <pinref part="IC1" gate="A" pin="IB"/>
-<wire x1="-40.64" y1="271.78" x2="-58.42" y2="271.78" width="0.1524" layer="91"/>
-<wire x1="-58.42" y1="271.78" x2="-58.42" y2="251.46" width="0.1524" layer="91"/>
+<wire x1="-40.64" y1="271.78" x2="-53.34" y2="271.78" width="0.1524" layer="91"/>
+<wire x1="-53.34" y1="271.78" x2="-53.34" y2="251.46" width="0.1524" layer="91"/>
 <pinref part="PIC" gate="G$1" pin="RB1"/>
-<wire x1="-58.42" y1="251.46" x2="-76.2" y2="251.46" width="0.1524" layer="91"/>
+<wire x1="-53.34" y1="251.46" x2="-76.2" y2="251.46" width="0.1524" layer="91"/>
 </segment>
 </net>
@@
 <segment>
 <pinref part="IC1" gate="A" pin="IC"/>
-<wire x1="-40.64" y1="269.24" x2="-60.96" y2="269.24" width="0.1524" layer="91"/>
-<wire x1="-60.96" y1="269.24" x2="-60.96" y2="254" width="0.1524" layer="91"/>
+<wire x1="-40.64" y1="269.24" x2="-55.88" y2="269.24" width="0.1524" layer="91"/>
+<wire x1="-55.88" y1="269.24" x2="-55.88" y2="254" width="0.1524" layer="91"/>
 <pinref part="PIC" gate="G$1" pin="RB2"/>
-<wire x1="-60.96" y1="254" x2="-76.2" y2="254" width="0.1524" layer="91"/>
+<wire x1="-55.88" y1="254" x2="-76.2" y2="254" width="0.1524" layer="91"/>
 </segment>
 </net>
@@
 <segment>
 <pinref part="IC1" gate="A" pin="ID"/>
-<wire x1="-40.64" y1="266.7" x2="-63.5" y2="266.7" width="0.1524" layer="91"/>
-<wire x1="-63.5" y1="266.7" x2="-63.5" y2="256.54" width="0.1524" layer="91"/>
+<wire x1="-40.64" y1="266.7" x2="-58.42" y2="266.7" width="0.1524" layer="91"/>
+<wire x1="-58.42" y1="266.7" x2="-58.42" y2="256.54" width="0.1524" layer="91"/>
 <pinref part="PIC" gate="G$1" pin="PGM/RB3"/>
-<wire x1="-63.5" y1="256.54" x2="-76.2" y2="256.54" width="0.1524" layer="91"/>
+<wire x1="-58.42" y1="256.54" x2="-76.2" y2="256.54" width="0.1524" layer="91"/>
 </segment>
 </net>
@@
 <segment>
 <pinref part="IC2" gate="A" pin="IA"/>
-<wire x1="-40.64" y1="236.22" x2="-66.04" y2="236.22" width="0.1524" layer="91"/>
-<wire x1="-66.04" y1="236.22" x2="-66.04" y2="259.08" width="0.1524" layer="91"/>
+<wire x1="-40.64" y1="236.22" x2="-60.96" y2="236.22" width="0.1524" layer="91"/>
+<wire x1="-60.96" y1="236.22" x2="-60.96" y2="259.08" width="0.1524" layer="91"/>
 <pinref part="PIC" gate="G$1" pin="RB4"/>
-<wire x1="-66.04" y1="259.08" x2="-76.2" y2="259.08" width="0.1524" layer="91"/>
+<wire x1="-60.96" y1="259.08" x2="-76.2" y2="259.08" width="0.1524" layer="91"/>
 </segment>
 </net>
@@
 <segment>
 <pinref part="IC2" gate="A" pin="IB"/>
-<wire x1="-40.64" y1="233.68" x2="-68.58" y2="233.68" width="0.1524" layer="91"/>
-<wire x1="-68.58" y1="233.68" x2="-68.58" y2="261.62" width="0.1524" layer="91"/>
+<wire x1="-40.64" y1="233.68" x2="-63.5" y2="233.68" width="0.1524" layer="91"/>
+<wire x1="-63.5" y1="233.68" x2="-63.5" y2="261.62" width="0.1524" layer="91"/>
 <pinref part="PIC" gate="G$1" pin="RB5"/>
-<wire x1="-68.58" y1="261.62" x2="-76.2" y2="261.62" width="0.1524" layer="91"/>
+<wire x1="-63.5" y1="261.62" x2="-76.2" y2="261.62" width="0.1524" layer="91"/>
 </segment>
 </net>
@@
 <segment>
 <pinref part="IC2" gate="A" pin="IC"/>
-<wire x1="-40.64" y1="231.14" x2="-71.12" y2="231.14" width="0.1524" layer="91"/>
-<wire x1="-71.12" y1="231.14" x2="-71.12" y2="264.16" width="0.1524" layer="91"/>
+<wire x1="-40.64" y1="231.14" x2="-66.04" y2="231.14" width="0.1524" layer="91"/>
+<wire x1="-66.04" y1="231.14" x2="-66.04" y2="264.16" width="0.1524" layer="91"/>
 <pinref part="PIC" gate="G$1" pin="PGC/RB6"/>
-<wire x1="-71.12" y1="264.16" x2="-76.2" y2="264.16" width="0.1524" layer="91"/>
+<wire x1="-66.04" y1="264.16" x2="-76.2" y2="264.16" width="0.1524" layer="91"/>
 </segment>
 </net>
@@
 <segment>
 <pinref part="IC2" gate="A" pin="ID"/>
-<wire x1="-40.64" y1="228.6" x2="-73.66" y2="228.6" width="0.1524" layer="91"/>
-<wire x1="-73.66" y1="228.6" x2="-73.66" y2="266.7" width="0.1524" layer="91"/>
+<wire x1="-40.64" y1="228.6" x2="-68.58" y2="228.6" width="0.1524" layer="91"/>
+<wire x1="-68.58" y1="228.6" x2="-68.58" y2="266.7" width="0.1524" layer="91"/>
 <pinref part="PIC" gate="G$1" pin="PGD/RB7"/>
-<wire x1="-73.66" y1="266.7" x2="-76.2" y2="266.7" width="0.1524" layer="91"/>
+<wire x1="-68.58" y1="266.7" x2="-76.2" y2="266.7" width="0.1524" layer="91"/>
 </segment>
 </net>
@@
 </segment>
 </net>
+<net name="RX" class="0">
+<segment>
+<pinref part="PIC" gate="G$1" pin="RX/RC7"/>
+<wire x1="-76.2" y1="233.68" x2="-73.66" y2="233.68" width="0.1524" layer="91"/>
+<label x="-73.66" y="233.68" size="1.778" layer="95"/>
+</segment>
+<segment>
+<pinref part="X2" gate="G$1" pin="3"/>
+<wire x1="-83.82" y1="193.04" x2="-88.9" y2="193.04" width="0.1524" layer="91"/>
+<label x="-88.9" y="193.04" size="1.778" layer="95" rot="R180"/>
+</segment>
+</net>
+<net name="TX" class="0">
+<segment>
+<pinref part="PIC" gate="G$1" pin="TX/RC6"/>
+<wire x1="-76.2" y1="231.14" x2="-73.66" y2="231.14" width="0.1524" layer="91"/>
+<label x="-73.66" y="231.14" size="1.778" layer="95"/>
+</segment>
+<segment>
+<pinref part="X2" gate="G$1" pin="2"/>
+<wire x1="-83.82" y1="195.58" x2="-88.9" y2="195.58" width="0.1524" layer="91"/>
+<label x="-88.9" y="195.58" size="1.778" layer="95" rot="R180"/>
+</segment>
+</net>

Commit message: Eagle
Parts:
- removed R1: (no value), rcl:R-EU_0207/10
- added JP1: (no value), pinhead:PINHD-1X3
- added R5: (no value), rcl:R-EU_0207/10
Connections:
- new net N$28: DIS2.DP, R5.1
- new net RC0: JP1.2, PIC.RC0/T1OSO
- new net RE0: PIC.RE0/!RD/AN5, R5.2
- net GND: now also JP1.3
- net VCC: now also JP1.1
Changed lines of the file:
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@@
 <part name="PIC" library="microchip" library_urn="urn:adsk.eagle:library:294" deviceset="PIC16F87*" device="P" package3d_urn="urn:adsk.eagle:package:20801/1" technology="7"/>
 <part name="Q1" library="special" library_urn="urn:adsk.eagle:library:367" deviceset="XTAL/S" device="" package3d_urn="urn:adsk.eagle:package:26647/2"/>
-<part name="R1" library="rcl" library_urn="urn:adsk.eagle:library:334" deviceset="R-EU_" device="0207/10" package3d_urn="urn:adsk.eagle:package:23491/2"/>
 <part name="C1" library="rcl" library_urn="urn:adsk.eagle:library:334" deviceset="C-EU" device="025-025X050" package3d_urn="urn:adsk.eagle:package:23629/2"/>
 <part name="C2" library="rcl" library_urn="urn:adsk.eagle:library:334" deviceset="C-EU" device="025-025X050" package3d_urn="urn:adsk.eagle:package:23629/2"/>
@@
 <part name="R4" library="rcl" library_urn="urn:adsk.eagle:library:334" deviceset="R-EU_" device="0207/10" package3d_urn="urn:adsk.eagle:package:23491/2"/>
 <part name="X2" library="con-subd" library_urn="urn:adsk.eagle:library:189" deviceset="F09" device="H" package3d_urn="urn:adsk.eagle:package:10276/1"/>
+<part name="R5" library="rcl" library_urn="urn:adsk.eagle:library:334" deviceset="R-EU_" device="0207/10" package3d_urn="urn:adsk.eagle:package:23491/2"/>
+<part name="JP1" library="pinhead" library_urn="urn:adsk.eagle:library:325" deviceset="PINHD-1X3" device="" package3d_urn="urn:adsk.eagle:package:22458/2"/>
 </parts>
 <sheets>
@@
 <attribute name="VALUE" x="-154.94" y="246.38" size="1.778" layer="96" rot="R270"/>
 </instance>
-<instance part="R1" gate="G$1" x="-152.4" y="274.32" smashed="yes">
-<attribute name="NAME" x="-156.21" y="275.8186" size="1.778" layer="95"/>
-<attribute name="VALUE" x="-156.21" y="271.018" size="1.778" layer="96"/>
-</instance>
 <instance part="C1" gate="G$1" x="-157.48" y="226.06" smashed="yes">
 <attribute name="NAME" x="-155.956" y="226.441" size="1.778" layer="95"/>
@@
 <attribute name="VALUE" x="-80.01" y="182.245" size="1.778" layer="96"/>
 <attribute name="NAME" x="-80.01" y="201.93" size="1.778" layer="95"/>
+</instance>
+<instance part="R5" gate="G$1" x="53.34" y="220.98" smashed="yes">
+<attribute name="NAME" x="49.53" y="222.4786" size="1.778" layer="95"/>
+<attribute name="VALUE" x="49.53" y="217.678" size="1.778" layer="96"/>
+</instance>
+<instance part="JP1" gate="A" x="10.16" y="198.12" smashed="yes">
+<attribute name="NAME" x="3.81" y="203.835" size="1.778" layer="95"/>
+<attribute name="VALUE" x="3.81" y="190.5" size="1.778" layer="96"/>
 </instance>
 </instances>
@@
 <label x="-88.9" y="187.96" size="1.778" layer="95" rot="R180"/>
 </segment>
+<segment>
+<pinref part="JP1" gate="A" pin="3"/>
+<wire x1="7.62" y1="195.58" x2="-2.54" y2="195.58" width="0.1524" layer="91"/>
+<label x="-2.54" y="195.58" size="1.778" layer="95"/>
+</segment>
 </net>
 <net name="VCC" class="0">
@@
 <junction x="-43.18" y="220.98"/>
 <label x="-43.18" y="218.44" size="1.778" layer="95" rot="R180"/>
+</segment>
+<segment>
+<pinref part="JP1" gate="A" pin="1"/>
+<wire x1="7.62" y1="200.66" x2="-2.54" y2="200.66" width="0.1524" layer="91"/>
+<label x="-2.54" y="200.66" size="1.778" layer="95"/>
 </segment>
 </net>
@@
 </segment>
 </net>
+<net name="N$28" class="0">
+<segment>
+<pinref part="DIS2" gate="N" pin="DP"/>
+<wire x1="43.18" y1="220.98" x2="48.26" y2="220.98" width="0.1524" layer="91"/>
+<pinref part="R5" gate="G$1" pin="1"/>
+</segment>
+</net>
+<net name="RE0" class="0">
+<segment>
+<pinref part="R5" gate="G$1" pin="2"/>
+<wire x1="58.42" y1="220.98" x2="60.96" y2="220.98" width="0.1524" layer="91"/>
+<label x="60.96" y="220.98" size="1.778" layer="95"/>
+</segment>
+<segment>
+<pinref part="PIC" gate="G$1" pin="RE0/!RD/AN5"/>
+<wire x1="-119.38" y1="248.92" x2="-121.92" y2="248.92" width="0.1524" layer="91"/>
+<label x="-121.92" y="248.92" size="1.778" layer="95" rot="R180"/>
+</segment>
+</net>
+<net name="RC0" class="0">
+<segment>
+<pinref part="JP1" gate="A" pin="2"/>
+<wire x1="7.62" y1="198.12" x2="-2.54" y2="198.12" width="0.1524" layer="91"/>
+<label x="-2.54" y="198.12" size="1.778" layer="95"/>
+</segment>
+<segment>
+<pinref part="PIC" gate="G$1" pin="RC0/T1OSO"/>
+<wire x1="-119.38" y1="233.68" x2="-121.92" y2="233.68" width="0.1524" layer="91"/>
+<label x="-121.92" y="233.68" size="1.778" layer="95" rot="R180"/>
+</segment>
+</net>
